File: Hardware Files/KitchenTimer.kicad_pcb (KiCad board)
At the start: 2 copper layers, 100 x 100 mm, 120 parts, among them J1 Conn_01x04, J2 USB_B_Micro, J3 Battery, Q1 P 1V 250uA 4A SOT-23, Q10 Q_NMOS_GSD, Q11 Q_NMOS_GSD, Q12 Q_NMOS_GSD, Q13 Q_NMOS_GSD, Q14 -30V 12A 14mΩ @ 8A, Q15 20V 7.5A 24mΩ @ 2.5Vgs, Q16 P 1V 250uA 4A SOT-23, Q17 P 1V 250uA 4A SOT-23, Q18 P 1V 250uA 4A SOT-23, Q19 P 1V 250uA 4A SOT-23, Q2 P 1V 250uA 4A SOT-23, Q20 P 1V 250uA 4A SOT-23, Q3 P 1V 250uA 4A SOT-23, Q4 P 1V 250uA 4A SOT-23, Q5 P 1V 250uA 4A SOT-23, Q6 Q_NMOS_GSD, Q7 Q_NMOS_GSD, Q8 Q_NMOS_GSD, Q9 Q_NMOS_GSD, SW1 SW_SPST, SW2 SW_SPST, SW3 SW_Push_Dual, SW4 SW_Push_Dual, SW5 SW_Push_Dual, SW6 SW_Push_Dual, U1 74HC595, U11 74HC595, U2 74HC595, U3 ESP-WROOM-02D, U4 AP34063S8G-13, U5 TP4056, U6 AP9101CK6, U7 NCP1117ST50T3G, U8 NCP1117ST33T3G, U9 74HC595

Commit message: update layout
Parts:
- removed C1, C2: 1uF, Capacitor_SMD:C_1206_3216Metric_Pad1.33x1.80mm_HandSolder
- removed LED1: SLR0564DBA4BD, KitchenTimer:SLR0564DBA4BD
- removed Q10, Q11, Q12, Q13, Q6, Q7, Q8, Q9: Q_NMOS_GSD, Package_TO_SOT_SMD:SOT-23
- removed R10, R11, R12, R13, R14, R6, R7, R8, R9: R, Resistor_SMD:R_0805_2012Metric_Pad1.20x1.40mm_HandSolder
- removed R17, R23, R24, R25, R26, R27, R28, R29, R30: 10k, Resistor_SMD:R_0805_2012Metric_Pad1.20x1.40mm_HandSolder
- removed U1, U2: 74HC595, Package_SO:SOIC-16_3.9x9.9mm_P1.27mm
- added C23: 1uF, Capacitor_SMD:C_1206_3216Metric_Pad1.33x1.80mm_HandSolder, B.Cu at (118.0, 11.0)
- added C24: 1uF, Capacitor_SMD:C_1206_3216Metric_Pad1.33x1.80mm_HandSolder, B.Cu at (118.0, 33.0)
- added R54: 10k, Resistor_SMD:R_0805_2012Metric_Pad1.20x1.40mm_HandSolder, B.Cu at (114.8, 11.6)
- added R55: 10k, Resistor_SMD:R_0805_2012Metric_Pad1.20x1.40mm_HandSolder, B.Cu at (117.4, 29.9)
- J1, SW1, SW2: moved to F.Cu
- moved J1 373.6 mm to (317.1, -233.5), turned to 270 degrees
- moved SW3 356.6 mm to (305.8, -189.5)
- moved SW4 356.6 mm to (316.8, -189.5)
- moved SW5 356.6 mm to (276.8, -189.5)
- moved SW6 356.6 mm to (287.8, -189.5)
- moved SW1 331.4 mm to (281.2, -227.8)
- moved U3 330.1 mm to (296.7, -222.8)
- moved C4 328.6 mm to (283.8, -233.8), turned to 180 degrees
- moved C3 328.3 mm to (283.8, -231.0), turned to 0 degrees
- moved SW2 325.9 mm to (277.5, -227.8)
- moved J2 293.1 mm to (341.5, -228.8)
- moved R49 164.6 mm to (280.5, -211.1)
- moved R51 164.6 mm to (280.5, -204.0)
- moved LED2 164.6 mm to (296.8, -204.0)
- moved R1 164.6 mm to (307.4, -206.5)
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Connections:
- U11 pad 10: Net-(U11-Pad10) -> !Clear
- U11 pad 11: Net-(U11-Pad11) -> Clock
- U11 pad 12: Net-(U11-Pad12) -> Latch
- U11 pad 13: Net-(U11-Pad13) -> ShiftRegister_Output_Enable
- U11 pad 14: Net-(U11-Pad14) -> Data
- U11 pad 16: Net-(U11-Pad16) -> +3V3
- U11 pad 8: Net-(U11-Pad8) -> GND
- U11 pad 9: Net-(U11-Pad9) -> ShiftRegister_1_overflow
- U9 pad 10: Net-(U9-Pad10) -> !Clear
- U9 pad 11: Net-(U9-Pad11) -> Clock
- U9 pad 12: Net-(U9-Pad12) -> Latch
- U9 pad 13: Net-(U9-Pad13) -> ShiftRegister_Output_Enable
- U9 pad 14: Net-(U9-Pad14) -> Data
- U9 pad 16: Net-(U9-Pad16) -> +3V3
- U9 pad 8: Net-(U9-Pad8) -> GND
- U9 pad 9: Net-(U9-Pad9) -> ShiftRegister_1_overflow
Routing:
- net BTN_StartStop: track 0.00 -> 92.8 mm, vias 0 -> 2
- net BTN_ResetCountdown: track 0.00 -> 90.0 mm
- net BTN_Down: track 0.00 -> 86.3 mm, vias 0 -> 3
- net Data: track 69.2 -> 133.0 mm, vias 2 -> 4
- net BTN_Up: track 0.00 -> 58.0 mm, vias 0 -> 2
- net Latch: track 71.4 -> 126.8 mm, vias 3 -> 5
- net ShiftRegister_Output_Enable: track 5.09 -> 55.8 mm, vias 0 -> 2
- net !Clear: track 48.4 -> 98.7 mm, vias 0 -> 2
- net Clock: track 61.7 -> 108.6 mm, vias 3 -> 5
- net ESP_RX: track 22.8 -> 50.7 mm, vias 0 -> 2
- net VDD: track 15.4 -> 40.2 mm, vias 0 -> 5
- net ESP_TX: track 19.9 -> 43.0 mm
- net ESP_Enable: track 0.00 -> 15.2 mm
- net +3V3: track 7.18 -> 14.3 mm, vias 0 -> 1
- net GND: track 0.00 -> 0.77 mm
- added copper zone on B.Cu, net GND
- added copper zone on F.Cu, net GND

Commit message: update layout
Parts:
- removed C5: 1uF, Capacitor_SMD:C_1206_3216Metric_Pad1.33x1.80mm_HandSolder
- removed Q1, Q2, Q3, Q4, Q5: P 1V 250uA 4A SOT-23, Package_TO_SOT_SMD:SOT-23
- removed R18, R19, R20, R21, R22: 10k, Resistor_SMD:R_0603_1608Metric_Pad0.98x0.95mm_HandSolder
- removed R31: 10k, Resistor_SMD:R_0805_2012Metric_Pad1.20x1.40mm_HandSolder
- C10, C7, C8, C9: footprint Capacitor_SMD:C_1206_3216Metric_Pad1.33x1.80mm_HandSolder -> Capacitor_SMD:C_0805_2012Metric_Pad1.18x1.45mm_HandSolder
- C12, C13, C15, C18, C19, C20, C21, C22, D1, D2, D3, J3, L1, Q14, Q15, R15, R16, R32, R37, R38, R39, R40, R41, R42, R43, R44, R45, R54, R55, U4, U5, U6, U7, U8: moved to F.Cu
- C23, C24, C6: footprint Capacitor_SMD:C_1206_3216Metric_Pad1.33x1.80mm_HandSolder -> Capacitor_SMD:C_0805_2012Metric_Pad1.18x1.45mm_HandSolder; moved to F.Cu
- moved U8 372.9 mm to (330.0, -229.2), turned to 0 degrees
- moved C20 343.3 mm to (322.2, -226.8), turned to 180 degrees
- moved C22 340.6 mm to (322.2, -229.5), turned to 180 degrees
- moved U5 320.1 mm to (205.3, -243.3), turned to 0 degrees
- moved D1 309.7 mm to (204.6, -235.0), turned to 0 degrees
- moved R37 308.1 mm to (207.1, -238.6), turned to 0 degrees
- moved C19 301.4 mm to (195.7, -238.4), turned to 0 degrees
- moved J3 300.6 mm to (181.6, -232.2), turned to 0 degrees
- moved C21 299.6 mm to (172.0, -220.3), turned to 0 degrees
- moved U4 298.4 mm to (191.4, -233.2), turned to 0 degrees
- moved Q15 297.3 mm to (180.2, -220.9), turned to 0 degrees
- moved L1 295.0 mm to (157.6, -239.3)
- moved D2 293.9 mm to (198.6, -231.7), turned to 0 degrees
- moved R39 291.5 mm to (197.9, -228.5), turned to 0 degrees
- moved Q14 288.1 mm to (196.9, -243.3), turned to 0 degrees
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Routing:
- net Char_1_Power: track 99.5 -> 4.84 mm
- net Net-(LED1-Pad12): track 73.9 -> 0.00 mm, vias 1 -> 0
- net Latch: track 126.8 -> 55.4 mm, vias 5 -> 2
- net Data: track 133.0 -> 63.8 mm, vias 4 -> 2
- net Net-(LED1-Pad9): track 67.7 -> 0.00 mm, vias 1 -> 0
- net Clock: track 108.6 -> 46.9 mm, vias 5 -> 2
- net LED_C: track 83.2 -> 21.6 mm
- net Char_2_Power: track 74.8 -> 15.1 mm, vias 4 -> 1
- net LED_F: track 66.1 -> 7.75 mm
- net Char_1: track 61.5 -> 4.36 mm
- net Net-(LED1-Pad4): track 53.6 -> 0.00 mm, vias 1 -> 0
- net Char_3_Power: track 69.8 -> 19.3 mm, vias 2 -> 1
- net LED_E: track 62.6 -> 13.3 mm
- net !Clear: track 98.7 -> 50.3 mm
- net Net-(LED1-Pad13): track 47.5 -> 0.00 mm, vias 1 -> 0
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- added copper zone on B.Cu, net +3V3
- removed copper zone on B.Cu, net GND

Commit message: update layout
Parts:
- J2: moved to F.Cu
- moved J2 18.4 mm to (327.0, -217.5), turned to 270 degrees
- moved C20 4.12 mm to (318.2, -225.8)
- moved C22 4.12 mm to (318.2, -228.5)
- moved U8 4.12 mm to (326.0, -228.2)

Commit message: update layout
Parts:
- removed C11, C14, C16, C17: 100uF ±20% 50V, Capacitor_SMD:CP_Elec_8x10.5
- removed C12, C15: 10uF ±10% 25V X5R, Capacitor_SMD:C_1206_3216Metric_Pad1.33x1.80mm_HandSolder
- removed C13: NP0 500V ±5% 100pF 1206, Capacitor_SMD:C_1206_3216Metric_Pad1.33x1.80mm_HandSolder
- removed C18: 100nF ±10% 50V X7R, Capacitor_SMD:C_1206_3216Metric_Pad1.33x1.80mm_HandSolder
- removed C19, C21: 220nF 50V, Capacitor_SMD:C_1206_3216Metric_Pad1.33x1.80mm_HandSolder
- removed D1: Orange LED, Diode_SMD:D_1206_3216Metric_Pad1.42x1.75mm_HandSolder
- removed D2: Green LED, Diode_SMD:D_1206_3216Metric_Pad1.42x1.75mm_HandSolder
- removed D3: 40V 3A 500mV@3A, Diode_SMD:D_SMB
- removed J3: Battery, .[--Stasis.Footprints.Library:WJ124-3.81-2P
- removed L1: 100µH 20% 1A, Inductor_SMD:L_Wuerth_HCI-1350
- removed Q14: -30V 12A 14mΩ @ 8A, .[--Stasis.Footprints.Library:SOP-8_3.9x4.9mm_P1.27mm
- removed Q15: 20V 7.5A 24mΩ @ 2.5Vgs, Package_SO:SOIC-8_3.9x4.9mm_P1.27mm
- removed R15, R16: 0R, Resistor_SMD:R_0805_2012Metric_Pad1.20x1.40mm_HandSolder
- removed R37: 0.3R, Resistor_SMD:R_0805_2012Metric_Pad1.20x1.40mm_HandSolder
- removed R38, R39, R55: 10k, Resistor_SMD:R_0805_2012Metric_Pad1.20x1.40mm_HandSolder
- removed R40: 180R, Resistor_SMD:R_0805_2012Metric_Pad1.20x1.40mm_HandSolder
- removed R41, R45: 1.2kΩ ±1% 0.25W, Resistor_SMD:R_0805_2012Metric_Pad1.20x1.40mm_HandSolder
- removed R42: 200k, Resistor_SMD:R_0805_2012Metric_Pad1.20x1.40mm_HandSolder
- removed R43: 47k, Resistor_SMD:R_0805_2012Metric_Pad1.20x1.40mm_HandSolder
- removed R44: 330R ±1% 0.25W, Resistor_SMD:R_0805_2012Metric_Pad1.20x1.40mm_HandSolder
- removed U4: AP34063S8G-13, Package_SO:SOIC-8_3.9x4.9mm_P1.27mm
- removed U5: TP4056, .[--Stasis.Footprints.Library:SOIC-8-1EP_3.9x4.9mm_P1.27mm_EP2.29x3mm
- removed U6: AP9101CK6, Package_TO_SOT_SMD:SOT-23-6_Handsoldering
- removed U7: NCP1117ST50T3G, Package_TO_SOT_SMD:SOT-223-3_TabPin2
- added C1: 10uF ±10% 25V X5R, Capacitor_SMD:C_1206_3216Metric_Pad1.33x1.80mm_HandSolder, F.Cu at (74.0, 31.8)
- added C2: 10uF ±10% 25V X5R, Capacitor_SMD:C_1206_3216Metric_Pad1.33x1.80mm_HandSolder, F.Cu at (74.0, 24.2)
- C23, C24, C6, R32, R54, U8: moved to B.Cu
- C3: footprint Capacitor_SMD:C_1206_3216Metric_Pad1.33x1.80mm_HandSolder -> Capacitor_SMD:C_0805_2012Metric_Pad1.18x1.45mm_HandSolder
- moved U8 358.7 mm to (74.2, 27.2), turned to 90 degrees
- moved SW1 355.3 mm to (34.5, 27.9)
- moved SW2 355.3 mm to (30.8, 27.9)
- moved R49 354.1 mm to (33.7, 42.9)
- moved R50 354.1 mm to (33.7, 46.4)
- moved R51 354.1 mm to (33.7, 50.0)
- moved R52 354.1 mm to (33.7, 57.1)
- moved R53 354.1 mm to (33.7, 53.6)
- moved C10 354.1 mm to (43.0, 63.2)
- moved C3 354.1 mm to (37.0, 23.0)
- moved C4 354.1 mm to (37.0, 20.2)
- moved C7 354.1 mm to (57.2, 63.2)
- moved C8 354.1 mm to (64.0, 63.3)
- moved C9 354.1 mm to (24.0, 63.2)
- moved J1 354.1 mm to (70.3, 20.5)
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Connections:
- C20 pad 1: SMPS_Output -> +5V
- U8 pad 3: SMPS_Output -> +5V
Routing:
- net ShiftRegister_1_overflow: track 0.00 -> 45.8 mm, vias 0 -> 2
- net GND: track 19.4 -> 64.6 mm, vias 2 -> 10
- net +3V3: track 57.5 -> 22.7 mm, vias 2 -> 5
- net +5V: track 0.00 -> 31.1 mm, vias 0 -> 1
- net ESP_Enable: track 15.2 -> 23.9 mm, vias 0 -> 1
- net BTN_ResetCountdown: track 94.2 -> 99.6 mm, vias 1 -> 3
- net SMPS_Output: track 3.12 -> 0.00 mm
- net BTN_Down: track 103.6 -> 105.8 mm
Other:
- board size 100 x 100 mm -> 72.5 x 56 mm

Commit message: add gnd connection
Routing:
- net GND: track 64.6 -> 72.4 mm, vias 10 -> 11
